Commit message: spawn in gazebo

File: leo/urdf/camera.xacro (robot description, xacro)
@@ -9,4 +9,9 @@
             <material name="orange"/>
         </visual>
+        <collision>
+            <geometry>
+                <box size="0.03 0.03 0.03"/>
+            </geometry>
+        </collision>
     </link>
     <link name="cam_linse">
@@ -17,9 +22,11 @@
             <material name="black"/>
         </visual>
+        <collision>
+            <geometry>
+                <cylinder radius="0.01" length="0.02"/>
+            </geometry>
+        </collision>
     </link>
     <link name="camera_link_optical"></link>
-    <gazebo reference="cam_linse">
-        <material>Gazebo/Black</material>
-    </gazebo>
     <joint name="cam_body_joint" type="fixed">
         <origin xyz="0.0 0.0 0.04" rpy="0.0 0.0 0.0"/>
@@ -38,4 +45,7 @@
     </joint>
     <!-- GAZEBO PLUGIN
+    <gazebo reference="cam_linse">
+        <material>Gazebo/Black</material>
+    </gazebo>
     <gazebo reference="cam">
         <material>Gazebo/Orange</material>

File: leo/urdf/chassi.xacro (robot description, xacro)
@@ -20,4 +20,10 @@
             <material name="black"/>
         </visual>
+        <collision>
+            <origin xyz="0.0 0.0 ${chassi_height/2}" rpy="0.0 0.0 0.0"/>
+            <geometry>
+                <box size="${chassi_length} ${chassi_width} ${chassi_height}"/>
+            </geometry>
+        </collision>
     </link>
     <link name="chassis_top">
@@ -29,4 +35,10 @@
             <material name="black"/>
         </visual>
+        <collision>
+            <origin xyz="0.0 0.0 ${chassi_top_height/2}" rpy="0.0 0.0 0.0"/>
+            <geometry>
+                <box size="${chassi_top_length} ${chassi_top_width} ${chassi_top_height}"/>
+            </geometry>
+        </collision>
     </link>
     <!-- WHEELS-->
@@ -40,4 +52,10 @@
                 <material name="white"/>
             </visual>
+            <collision>
+                <origin xyz="0.0 0.0 0.0" rpy="${pi/2} 0.0 0.0"/>
+                <geometry>
+                    <cylinder radius="${wheel_radius}" length="${wheel_length}"/>
+                </geometry>
+            </collision>
         </link>
     </xacro:macro>

File: leo/urdf/leopard.urdf.xacro (robot description, xacro)
@@ -4,7 +4,7 @@
     <xacro:include filename="chassi.xacro"/>
     <xacro:include filename="joints.xacro"/>
-    <xacro:include filename="turret.xacro"/> <!--
+    <xacro:include filename="turret.xacro"/> <!-- -->
     <xacro:include filename="pipe.xacro"/>
     <xacro:include filename="lidar.xacro"/>
-    <xacro:include filename="camera.xacro"/> -->
+    <xacro:include filename="camera.xacro"/>
 </robot>

File: leo/urdf/lidar.xacro (robot description, xacro)
@@ -9,4 +9,9 @@
             <material name="orange" />
         </visual>
+        <collision>
+            <geometry>
+                <box size="0.03 0.03 0.03" />
+            </geometry>
+        </collision>
     </link>
     <link name="laser_frame">
@@ -18,4 +23,10 @@
             <material name="black" />
         </visual>
+        <collision>
+            <origin xyz="0.0 0.0 0.0" rpy="0.0 0.0 ${pi/2}"/>
+            <geometry>
+                <cylinder radius="0.035" length="0.02" />
+            </geometry>
+        </collision>
     </link>
     <joint name="laser_joint" type="fixed">

File: leo/urdf/material.xacro (robot description, xacro)
@@ -22,3 +22,30 @@
         <color rgba="1 1 0 1"/>
     </material>
+    <xacro:macro name="box_inertia" params="m l w h xyz rpy">
+        <inertial>
+            <origin xyz="${xyz}" rpy="${rpy}" />
+            <mass value="${m}" />
+            <inertia ixx="${(m/12) * (h*h + l*l)}" ixy="0" ixz="0"
+                     iyy="${(m/12) * (w*w + l*l)}" iyz="0"
+                     izz="${(m/12) * (w*w + h*h)}" />
+        </inertial>
+    </xacro:macro>
+    <xacro:macro name="cylinder_inertia" params="m r h xyz rpy">
+        <inertial>
+            <origin xyz="${xyz}" rpy="${rpy}" />
+            <mass value="${m}" />
+            <inertia ixx="${(m/12) * (3*r*r + h*h)}" ixy="0" ixz="0"
+                     iyy="${(m/12) * (3*r*r + h*h)}" iyz="0"
+                     izz="${(m/2) * (r*r)}" />
+        </inertial>
+    </xacro:macro>
+    <xacro:macro name="sphere_inertia" params="m r xyz rpy">
+        <inertial>
+            <origin xyz="${xyz}" rpy="${rpy}" />
+            <mass value="${m}" />
+            <inertia ixx="${(2/5) * m * r * r}" ixy="0" ixz="0"
+                     iyy="${(2/5) * m * r * r}" iyz="0"
+                     izz="${(2/5) * m * r * r}" />
+        </inertial>
+    </xacro:macro>
 </robot>

File: leo/urdf/pipe.xacro (robot description, xacro)
@@ -9,4 +9,9 @@
             <material name="white" />
         </visual>
+        <collision>
+            <geometry>
+                <box size="0.08 0.04 0.05" />
+            </geometry>
+        </collision>
     </link>
     <link name="gun_deko">
@@ -18,4 +23,10 @@
             <material name="white" />
         </visual>
+        <collision>
+            <origin xyz="0.0 0.0 0.0" rpy="0.0 ${pi/4} 0.0" />
+            <geometry>
+                <box size="0.036 0.04 0.036" />
+            </geometry>
+        </collision>
     </link>
     <link name="gun_pipe">
@@ -27,4 +38,10 @@
             <material name="white" />
         </visual>
+        <collision>
+            <origin xyz="0.15 0.0 0.0" rpy="0.0 ${pi/2} 0.0" />
+            <geometry>
+                <cylinder radius="0.009" length="0.3" />
+            </geometry>
+        </collision>
     </link>
     <!-- Gun_joint -->

File: leo/urdf/turret.xacro (robot description, xacro)
@@ -10,4 +10,9 @@
                 <material name="yellow" />
             </visual>
+            <collision>
+                <geometry>
+                    <cylinder radius="0.06" length="0.005" />
+                </geometry>
+            </collision>
         </link>
     </xacro:macro>
@@ -22,4 +27,10 @@
             <material name="white" />
         </visual>
+        <collision>
+            <geometry>
+                <box size="0.28 0.17 0.05" />
+            </geometry>
+            <material name="white" />
+        </collision>
     </link>
     <xacro:macro name="turm_seite" params="prefix">
@@ -31,8 +42,13 @@
                 <material name="white" />
             </visual>
+            <collision>
+                <geometry>
+                    <box size="0.1 0.05 0.05" />
+                </geometry>
+            </collision>
         </link>
     </xacro:macro>
-    <xacro:turm_seite prefix="r"/>
-    <xacro:turm_seite prefix="l"/>
+    <xacro:turm_seite prefix="r" />
+    <xacro:turm_seite prefix="l" />
     <!-- JOINTS Turret -->
     <joint name="fixirung" type="fixed">
@@ -50,7 +66,7 @@
         <parent link="down_coil" />
         <child link="top_coil" />
-        <axis xyz="0 0 1"/>
-        <limit lower="-${pi*2}" upper="${pi*2}" velocity="1.0" effort="10.0"/>
-        <origin xyz="0 0 0.005" rpy="0 0 0"/>
+        <axis xyz="0 0 1" />
+        <limit lower="-${pi*2}" upper="${pi*2}" velocity="1.0" effort="10.0" />
+        <origin xyz="0 0 0.005" rpy="0 0 0" />
     </joint>
     <!-- Turm_joints-->

Commit message: added Gazebo Colors

File: leo/urdf/camera.xacro (robot description, xacro)
@@ -32,5 +32,5 @@
                            xyz="0 0 0" rpy="0 0 0"/>
     </link>
-    <link name="camera_link_optical"></link>
+    <link name="leo_optic"></link>
     <joint name="cam_body_joint" type="fixed">
         <origin xyz="0.0 0.0 0.04" rpy="0.0 0.0 0.0"/>
@@ -43,10 +43,10 @@
         <child link="cam_linse"/>
     </joint>
-    <joint name="camera_optical_joint" type="fixed">
+    <joint name="leo_optic_joint" type="fixed">
         <origin xyz="0 0.0 0.0" rpy="${-pi/2} 0.0 ${-pi/2}"/>
         <parent link="cam"/>
-        <child link="camera_link_optical"/>
+        <child link="leo_optic"/>
     </joint>
-    <!-- GAZEBO PLUGIN
+    <!-- GAZEBO PLUGIN -->
     <gazebo reference="cam_linse">
         <material>Gazebo/Black</material>
@@ -54,4 +54,5 @@
     <gazebo reference="cam">
         <material>Gazebo/Orange</material>
+    <!--
         <sensor name="camera" type="camera">
             <pose> 0 0 0 0 0 0 </pose>
@@ -71,7 +72,7 @@
             </camera>
             <plugin name="camera_controller" filename="libgazebo_ros_camera.so">
-                <frame_name>camera_link_optical</frame_name>
+                <frame_name>leo_optic</frame_name>
             </plugin>
-        </sensor>
-    </gazebo> -->
+        </sensor> -->
+    </gazebo>
 </robot>

File: leo/urdf/chassi.xacro (robot description, xacro)
@@ -29,4 +29,7 @@
                            xyz="0.0 0.0 ${chassi_height/2}" rpy="0 0 0"/>
     </link>
+    <gazebo reference="chassis">
+        <material>Gazebo/Grass</material>
+    </gazebo>
     <link name="chassis_top">
         <visual>
@@ -46,4 +49,7 @@
                            xyz="0.0 0.0 ${chassi_top_height/2}" rpy="0 0 0"/>
     </link>
+    <gazebo reference="chassis_top">
+        <material>Gazebo/Grass</material>
+    </gazebo>
     <!-- WHEELS-->
     <xacro:macro name="wheel_link" params="prefix ">
@@ -65,4 +71,7 @@
                            xyz="0 0 0" rpy="${pi/2} 0.0 0.0"/>
         </link>
+        <gazebo reference="${prefix}_wheel">
+            <material>Gazebo/Grey</material>
+        </gazebo>
     </xacro:macro>
     <xacro:wheel_link prefix="right"/>

File: leo/urdf/lidar.xacro (robot description, xacro)
@@ -17,4 +17,7 @@
                            xyz="0 0 0" rpy="0 0 0"/>
     </link>
+    <gazebo reference="lidar_mount">
+        <material>Gazebo/Grass</material>
+    </gazebo>
     <link name="laser_frame">
         <visual>
@@ -34,4 +37,7 @@
                            xyz="0 0 0" rpy="0 0 ${pi/2}"/>
     </link>
+    <gazebo reference="laser_frame">
+        <material>Gazebo/Black</material>
+    </gazebo>
     <joint name="laser_joint" type="fixed">
         <parent link="lidar_mount" />

File: leo/urdf/pipe.xacro (robot description, xacro)
@@ -17,4 +17,7 @@
                            xyz="0 0 0" rpy="0 0 0"/>
     </link>
+    <gazebo reference="turm_gun">
+        <material>Gazebo/Grass</material>
+    </gazebo>
     <link name="gun_deko">
         <visual>
@@ -34,4 +37,7 @@
                            xyz="0 0 0" rpy="0.0 ${pi/4} 0.0"/>
     </link>
+    <gazebo reference="gun_deko">
+        <material>Gazebo/Grass</material>
+    </gazebo>
     <link name="gun_pipe">
         <visual>
@@ -40,5 +46,5 @@
                 <cylinder radius="0.009" length="0.3" />
             </geometry>
-            <material name="white" />
+            <material name="red" />
         </visual>
         <collision>
@@ -51,4 +57,27 @@
                            xyz="0.15 0.0 0.0" rpy="0.0 ${pi/2} 0.0"/>
     </link>
+    <gazebo reference="gun_pipe">
+        <material>Gazebo/Red</material>
+    </gazebo>
+    <link name="gun_pipe_tail">
+        <visual>
+            <origin xyz="0.0 0.0 0.0" rpy="0.0 ${pi/2} 0.0" />
+            <geometry>
+                <cylinder radius="0.0075" length="0.001" />
+            </geometry>
+            <material name="black" />
+        </visual>
+        <collision>
+            <origin xyz="0.0 0.0 0.0" rpy="0.0 ${pi/2} 0.0" />
+            <geometry>
+                <cylinder radius="0.0075" length="0.001" />
+            </geometry>
+        </collision>
+        <xacro:cylinder_inertia m="0.001" r="0.00759" h="0.001"
+                           xyz="0.0 0.0 0.0" rpy="0.0 ${pi/2} 0.0"/>
+    </link>
+    <gazebo reference="gun_pipe_tail">
+        <material>Gazebo/Black</material>
+    </gazebo>
     <!-- Gun_joint -->
     <joint name="joint_4" type="revolute">
@@ -69,3 +98,8 @@
         <origin xyz="0.0 0.0 0.0" rpy="0.0 0.0 0.0" />
     </joint>
+    <joint name="gun_rohr_deko" type="fixed">
+        <parent link="gun_pipe" />
+        <child link="gun_pipe_tail" />
+        <origin xyz="0.3005 0.0 0.0" rpy="0.0 0.0 0.0" />
+    </joint>
 </robot>

File: leo/urdf/turret.xacro (robot description, xacro)
@@ -38,4 +38,7 @@
                            xyz="0 0 0" rpy="0 0 0"/>
     </link>
+    <gazebo reference="turm_top_">
+        <material>Gazebo/Grass</material>
+    </gazebo>
     <xacro:macro name="turm_seite" params="prefix">
         <link name="turm_top_${prefix}">
@@ -54,4 +57,32 @@
                            xyz="0 0 0" rpy="0 0 0"/>
         </link>
+        <gazebo reference="turm_top_${prefix}">
+            <material>Gazebo/Grass</material>
+        </gazebo>
+        <link name="turm_deko_${prefix}">
+            <visual>
+                <origin xyz="0.0 0.0 0.0" rpy="0.0 ${pi/4} 0.0" />
+                <geometry>
+                    <box size="0.0355 0.05 0.0355" />
+                </geometry>
+                <material name="white" />
+            </visual>
+            <collision>
+                <origin xyz="0.0 0.0 0.0" rpy="0.0 ${pi/4} 0.0" />
+                <geometry>
+                    <box size="0.0355 0.05 0.0355" />
+                </geometry>
+            </collision>
+            <xacro:box_inertia m="0.1" l="0.0355" w="0.05" h="0.0355"
+                               xyz="0 0 0" rpy="0.0 ${pi/4} 0.0"/>
+        </link>
+        <gazebo reference="turm_deko_${prefix}">
+            <material>Gazebo/Grass</material>
+        </gazebo>
+        <joint name="gun_deko_${prefix}" type="fixed">
+            <parent link="turm_top_${prefix}" />
+            <child link="turm_deko_${prefix}" />
+            <origin xyz="0.05 0.0 0.0" rpy="0.0 0.0 0.0" />
+        </joint>
     </xacro:macro>
     <xacro:turm_seite prefix="r" />

Commit message: added cam and Lidar for Gazebo

File: leo/urdf/camera.xacro (robot description, xacro)
@@ -54,5 +54,4 @@
     <gazebo reference="cam">
         <material>Gazebo/Orange</material>
-    <!--
         <sensor name="camera" type="camera">
             <pose> 0 0 0 0 0 0 </pose>
@@ -74,5 +73,5 @@
                 <frame_name>leo_optic</frame_name>
             </plugin>
-        </sensor> -->
+        </sensor>
     </gazebo>
 </robot>

File: leo/urdf/lidar.xacro (robot description, xacro)
@@ -15,5 +15,5 @@
         </collision>
         <xacro:box_inertia m="0.02" l="0.03" w="0.03" h="0.03"
-                           xyz="0 0 0" rpy="0 0 0"/>
+            xyz="0 0 0" rpy="0 0 0" />
     </link>
     <gazebo reference="lidar_mount">
@@ -22,5 +22,5 @@
     <link name="laser_frame">
         <visual>
-            <origin xyz="0.0 0.0 0.0" rpy="0.0 0.0 ${pi/2}"/>
+            <origin xyz="0.0 0.0 0.0" rpy="0.0 0.0 ${pi/2}" />
             <geometry>
                 <cylinder radius="0.035" length="0.02" />
@@ -29,5 +29,5 @@
         </visual>
         <collision>
-            <origin xyz="0.0 0.0 0.0" rpy="0.0 0.0 ${pi/2}"/>
+            <origin xyz="0.0 0.0 0.0" rpy="0.0 0.0 ${pi/2}" />
             <geometry>
                 <cylinder radius="0.035" length="0.02" />
@@ -35,8 +35,35 @@
         </collision>
         <xacro:cylinder_inertia m="0.01" r="0.035" h="0.02"
-                           xyz="0 0 0" rpy="0 0 ${pi/2}"/>
+            xyz="0 0 0" rpy="0 0 ${pi/2}" />
     </link>
     <gazebo reference="laser_frame">
         <material>Gazebo/Black</material>
+        <sensor name="laser" type="ray">
+            <pose> 0 0 0 0 0 0 </pose>
+            <visualize>true</visualize>
+            <update_rate>10</update_rate>
+            <ray>
+                <scan>
+                    <horizontal>
+                        <samples>360</samples>
+                        <resolution>1</resolution>
+                        <min_angle>0.00</min_angle>
+                        <max_angle>3.14</max_angle>
+                    </horizontal>
+                </scan>
+                <range>
+                    <min>0.3</min>
+                    <max>6</max>
+                </range>
+            </ray>
+            <plugin name="laser_controller" filename="libgazebo_ros_ray_sensor.so">
+                <ros>
+                    <argument>--ros-args --remap ~/out:=scan</argument> <!-- - -ros-args - -remap
+                    ~/out:=scan -->
+                </ros>
+                <output_type>sensor_msgs/LaserScan</output_type>
+                <frame_name>laser_frame</frame_name>
+            </plugin>
+        </sensor>
     </gazebo>
     <joint name="laser_joint" type="fixed">
