Commit message: lidar and cam for gz ready

File: leo/urdf/gazebo.xacro (robot description, xacro)
@@ -24,4 +24,26 @@
             <robot_base_frame>base_footprint</robot_base_frame>
         </plugin>
+        <plugin name="gazebo_ros_diff_drive" filename="libgazebo_ros_diff_drive.so">
+            <!-- Update rate in Hz -->
+            <update_rate>50</update_rate>
+            <!-- wheels -->
+            <left_joint>joint_3</left_joint>
+            <right_joint>joint_4</right_joint>
+            <!-- kinematics -->
+            <wheel_separation>1.25</wheel_separation>
+            <wheel_diameter>0.6</wheel_diameter>
+            <!-- limits -->
+            <max_wheel_torque>20</max_wheel_torque>
+            <max_wheel_acceleration>1.0</max_wheel_acceleration>
+            <!-- input -->
+            <command_topic>turm/cmd_vel</command_topic>
+            <!-- output -->
+            <publish_odom>true</publish_odom>
+            <publish_odom_tf>true</publish_odom_tf>
+            <publish_wheel_tf>true</publish_wheel_tf>
+            <odometry_topic>odom</odometry_topic>
+            <odometry_frame>odom</odometry_frame>
+            <robot_base_frame>base_footprint</robot_base_frame>
+        </plugin>
     </gazebo>
 </robot>

File: leo/urdf/lidar.xacro (robot description, xacro)
@@ -70,5 +70,5 @@
         <parent link="lidar_mount" />
         <child link="laser_frame" />
-        <origin xyz="0.0 0.0 0.02" rpy="0.0 0.0 0.0" />
+        <origin xyz="0.0 0.0 0.02" rpy="0.0 0.0 ${-pi/2}" />
     </joint>
     <joint name="lidar_mount_joint" type="fixed">
@@ -77,36 +77,3 @@
         <child link="lidar_mount" />
     </joint>
-    <!-- GAZEBO PLUGINS
-        <gazebo reference="laser_frame">
-            <material>Gazebo/Black</material>
-        </gazebo>
-        <gazebo reference="laser_frame">
-            <material>Gazebo/Black</material>
-            <sensor name="laser" type="ray">
-                <pose> 0 0 0 0 0 0 </pose>
-                <visualize>true</visualize>
-                <update_rate>10</update_rate>
-                <ray>
-                    <scan>
-                        <horizontal>
-                            <samples>360</samples>
-                            <resolution>1</resolution>
-                            <min_angle>0.00</min_angle>
-                            <max_angle>3.14</max_angle>
-                        </horizontal>
-                    </scan>
-                    <range>
-                        <min>0.3</min>
-                        <max>6</max>
-                    </range>
-                </ray>
-                <plugin name="laser_controller" filename="libgazebo_ros_ray_sensor.so">
-                    <ros>
-                        <argument>- -ros-args - -remap ~/out:=scan</argument> <!- - - -ros-args - -remap ~/out:=scan - ->
-                    </ros>
-                    <output_type>sensor_msgs/LaserScan</output_type>
-                    <frame_name>laser_frame</frame_name>
-                </plugin>
-            </sensor>
-        </gazebo> -->
 </robot>
