Commit message: changed 2 joints to fixed but does not work

File: leo/urdf/chassi.xacro (robot description, xacro)
@@ -73,6 +73,6 @@
         <gazebo reference="${prefix}_wheel">
             <material>Gazebo/Grey</material>
-            <mu1 value="0.001"/>
-            <mu2 value="0.001"/>
+            <mu1 value="0.1"/>
+            <mu2 value="0.1"/>
         </gazebo>
     </xacro:macro>

File: leo/urdf/pipe.xacro (robot description, xacro)
@@ -81,4 +81,5 @@
     </gazebo>
     <!-- Gun_joint -->
+<!--
     <joint name="joint_4" type="revolute">
         <parent link="turm_top_" />
@@ -86,4 +87,9 @@
         <axis xyz="0 -1 0" />
         <limit lower="-0.05" upper="0.4" velocity="50.0" effort="1000.0" />
+        <origin xyz="0.18 0 0" rpy="0 0 0" />
+    </joint> -->
+    <joint name="joint_4" type="fixed">
+        <parent link="turm_top_" />
+        <child link="turm_gun" />
         <origin xyz="0.18 0 0" rpy="0 0 0" />
     </joint>

File: leo/urdf/ros2_control.xacro (robot description, xacro)
@@ -28,21 +28,21 @@
         </plugin>
     </gazebo>
-    <!-- Plugin 2 für Turm und Kanone-->
+    <!-- Plugin 2 für Turm und Kanone
     <gazebo>
         <plugin name="gazebo_ros_diff_drive" filename="libgazebo_ros_diff_drive.so">
-            <!-- Update rate in Hz -->
+            <!- - Update rate in Hz - ->
             <update_rate>50</update_rate>
-            <!-- wheels -->
+            <!- - wheels - ->
             <left_joint>joint_3</left_joint>
             <right_joint>joint_4</right_joint>
-            <!-- kinematics -->
+            <!- - kinematics - ->
             <wheel_separation>1.25</wheel_separation>
             <wheel_diameter>0.6</wheel_diameter>
-            <!-- limits -->
+            <!- - limits - ->
             <max_wheel_torque>20</max_wheel_torque>
             <max_wheel_acceleration>1.0</max_wheel_acceleration>
-            <!-- input -->
+            <!- - input - ->
             <command_topic>turm/cmd_vel</command_topic>
-            <!-- output -->
+            <!- - output - ->
             <publish_odom>true</publish_odom>
             <publish_odom_tf>true</publish_odom_tf>
@@ -53,3 +53,4 @@
         </plugin>
     </gazebo>
+-->
 </robot>

File: leo/urdf/turret.xacro (robot description, xacro)
@@ -94,10 +94,11 @@
         <child link="down_coil" />
     </joint>
-    <!-- change to moving if - joint für den turm
+    <!-- change to moving if - joint für den turm -->
     <joint name="turret_coil_joint" type="fixed">
         <origin xyz="0.0 0.0 0.005" rpy="0.0 0.0 0.0" />
         <parent link="down_coil" />
         <child link="top_coil" />
-    </joint>  -->
+    </joint>
+<!--
     <joint name="joint_3" type="revolute">
         <parent link="down_coil" />
@@ -106,5 +107,5 @@
         <limit lower="-${pi*2}" upper="${pi*2}" velocity="1.0" effort="10.0" />
         <origin xyz="0 0 0.005" rpy="0 0 0" />
-    </joint>
+    </joint> -->
     <!-- Turm_joints-->
     <joint name="turm_top_joint" type="fixed">
