Commit message: unbreak gazebo

File: leo/urdf/leopard.urdf.xacro (robot description, xacro)
@@ -1,13 +1,21 @@
 <?xml version="1.0"?>
 <robot xmlns:xacro="http://www.ros.org/wiki/xacro" name="leo">
-    <xacro:include filename="material.xacro"/>
-    <xacro:include filename="chassi.xacro"/>
-    <xacro:include filename="joints.xacro"/>
-    <xacro:include filename="turret.xacro"/>
-   <!--
+  <xacro:arg name="use_ros2_control" default="true"/>
+  <xacro:arg name="sim_mode" default="false"/>
+  <xacro:include filename="material.xacro"/>
+  <xacro:include filename="chassi.xacro"/>
+  <xacro:include filename="joints.xacro"/>
+  <xacro:include filename="turret.xacro"/>
+  <xacro:if value="$(arg use_ros2_control)">
+    <xacro:include filename="ros2_control.xacro"/>
+  </xacro:if>
+  <xacro:unless value="$(arg use_ros2_control)">
+    <xacro:include filename="gazebo.xacro"/>
+  </xacro:unless>
+  <xacro:include filename="lidar.xacro"/>
+  <xacro:include filename="camera.xacro"/>
+  <!--
     <xacro:include filename="pipe.xacro"/>
-    <xacro:include filename="lidar.xacro"/> -->
-    <xacro:include filename="camera.xacro"/>
-  <!--  <xacro:include filename="gazebo.xacro"/> -->
-    <xacro:include filename="ros2_control.xacro"/>
+    -->
+  <!--   -->
 </robot>

File: leo/urdf/ros2_control.xacro (robot description, xacro)
@@ -1,33 +1,36 @@
 <?xml version="1.0"?>
 <robot xmlns:xacro="http://www.ros.org/wiki/xacro">
-    <ros2_control name="RealRobot" type="system">
-        <hardware>
-            <plugin>diffdrive_arduino/DiffDriveArduino</plugin>
-            <param name="left_wheel_name">joint_2</param>
-            <param name="right_wheel_name">joint_1</param>
-            <param name="loop_rate">30</param>
-            <param name="device">/dev/ttyUSB0</param>
-            <param name="baud_rate">57600</param>
-            <param name="timeout">1000</param>
-            <param name="enc_counts_per_rev">473</param>
-        </hardware>
-        <joint name="joint_1">
-            <command_interface name="velocity">
-                <param name="min">-10</param>
-                <param name="max">10</param>
-            </command_interface>
-            <state_interface name="velocity" />
-            <state_interface name="position" />
-        </joint>
-        <joint name="joint_2">
-            <command_interface name="velocity">
-                <param name="min">-10</param>
-                <param name="max">10</param>
-            </command_interface>
-            <state_interface name="velocity" />
-            <state_interface name="position" />
-        </joint>
-    </ros2_control>
-<!--    <ros2_control name="GazeboSystem" type="system">
+    <xacro:unless value="$(arg sim_mode)">
+        <ros2_control name="RealRobot" type="system">
+            <hardware>
+                <plugin>diffdrive_arduino/DiffDriveArduino</plugin>
+                <param name="left_wheel_name">joint_2</param>
+                <param name="right_wheel_name">joint_1</param>
+                <param name="loop_rate">30</param>
+                <param name="device">/dev/ttyUSB0</param>
+                <param name="baud_rate">57600</param>
+                <param name="timeout">1000</param>
+                <param name="enc_counts_per_rev">473</param>
+            </hardware>
+            <joint name="joint_1">
+                <command_interface name="velocity">
+                    <param name="min">-10</param>
+                    <param name="max">10</param>
+                </command_interface>
+                <state_interface name="velocity" />
+                <state_interface name="position" />
+            </joint>
+            <joint name="joint_2">
+                <command_interface name="velocity">
+                    <param name="min">-10</param>
+                    <param name="max">10</param>
+                </command_interface>
+                <state_interface name="velocity" />
+                <state_interface name="position" />
+            </joint>
+        </ros2_control>
+    </xacro:unless>
+    <xacro:if value="$(arg sim_mode)">
+        <ros2_control name="GazeboSystem" type="system">
         <hardware>
             <plugin>gazebo_ros2_control/GazeboSystem</plugin>
@@ -49,5 +52,6 @@
             <state_interface name="position" />
         </joint>
-    </ros2_control> -->
+    </ros2_control>
+</xacro:if>
     <gazebo>
         <plugin name="gazebo_ros2_control" filename="libgazebo_ros2_control.so">

Commit message: backup loaded

File: leo/urdf/leopard.urdf.xacro (robot description, xacro)
@@ -1,21 +1,13 @@
 <?xml version="1.0"?>
 <robot xmlns:xacro="http://www.ros.org/wiki/xacro" name="leo">
-  <xacro:arg name="use_ros2_control" default="true"/>
-  <xacro:arg name="sim_mode" default="false"/>
-  <xacro:include filename="material.xacro"/>
-  <xacro:include filename="chassi.xacro"/>
-  <xacro:include filename="joints.xacro"/>
-  <xacro:include filename="turret.xacro"/>
-  <xacro:if value="$(arg use_ros2_control)">
+    <xacro:include filename="material.xacro"/>
+    <xacro:include filename="chassi.xacro"/>
+    <xacro:include filename="joints.xacro"/>
+    <xacro:include filename="turret.xacro"/>
+    <!--
+    <xacro:include filename="pipe.xacro"/> -->
+    <xacro:include filename="lidar.xacro"/>
+    <xacro:include filename="camera.xacro"/>
+  <!--  <xacro:include filename="gazebo.xacro"/> -->
     <xacro:include filename="ros2_control.xacro"/>
-  </xacro:if>
-  <xacro:unless value="$(arg use_ros2_control)">
-    <xacro:include filename="gazebo.xacro"/>
-  </xacro:unless>
-  <xacro:include filename="lidar.xacro"/>
-  <xacro:include filename="camera.xacro"/>
-  <!--
-    <xacro:include filename="pipe.xacro"/>
-    -->
-  <!--   -->
 </robot>

File: leo/urdf/ros2_control.xacro (robot description, xacro)
@@ -1,36 +1,33 @@
 <?xml version="1.0"?>
 <robot xmlns:xacro="http://www.ros.org/wiki/xacro">
-    <xacro:unless value="$(arg sim_mode)">
-        <ros2_control name="RealRobot" type="system">
-            <hardware>
-                <plugin>diffdrive_arduino/DiffDriveArduino</plugin>
-                <param name="left_wheel_name">joint_2</param>
-                <param name="right_wheel_name">joint_1</param>
-                <param name="loop_rate">30</param>
-                <param name="device">/dev/ttyUSB0</param>
-                <param name="baud_rate">57600</param>
-                <param name="timeout">1000</param>
-                <param name="enc_counts_per_rev">473</param>
-            </hardware>
-            <joint name="joint_1">
-                <command_interface name="velocity">
-                    <param name="min">-10</param>
-                    <param name="max">10</param>
-                </command_interface>
-                <state_interface name="velocity" />
-                <state_interface name="position" />
-            </joint>
-            <joint name="joint_2">
-                <command_interface name="velocity">
-                    <param name="min">-10</param>
-                    <param name="max">10</param>
-                </command_interface>
-                <state_interface name="velocity" />
-                <state_interface name="position" />
-            </joint>
-        </ros2_control>
-    </xacro:unless>
-    <xacro:if value="$(arg sim_mode)">
-        <ros2_control name="GazeboSystem" type="system">
+    <ros2_control name="RealRobot" type="system">
+        <hardware>
+            <plugin>diffdrive_arduino/DiffDriveArduino</plugin>
+            <param name="left_wheel_name">joint_2</param>
+            <param name="right_wheel_name">joint_1</param>
+            <param name="loop_rate">30</param>
+            <param name="device">/dev/ttyUSB0</param>
+            <param name="baud_rate">57600</param>
+            <param name="timeout">1000</param>
+            <param name="enc_counts_per_rev">473</param>
+        </hardware>
+        <joint name="joint_1">
+            <command_interface name="velocity">
+                <param name="min">-10</param>
+                <param name="max">10</param>
+            </command_interface>
+            <state_interface name="velocity" />
+            <state_interface name="position" />
+        </joint>
+        <joint name="joint_2">
+            <command_interface name="velocity">
+                <param name="min">-10</param>
+                <param name="max">10</param>
+            </command_interface>
+            <state_interface name="velocity" />
+            <state_interface name="position" />
+        </joint>
+    </ros2_control>
+<!--    <ros2_control name="GazeboSystem" type="system">
         <hardware>
             <plugin>gazebo_ros2_control/GazeboSystem</plugin>
@@ -52,6 +49,5 @@
             <state_interface name="position" />
         </joint>
-    </ros2_control>
-</xacro:if>
+    </ros2_control> -->
     <gazebo>
         <plugin name="gazebo_ros2_control" filename="libgazebo_ros2_control.so">
