Commit message: in work

File: tank_description/urdf/chassi.xacro (robot description, xacro)
@@ -47,5 +47,5 @@
         </collision>
         <xacro:box_inertia m="1.0" l="${chassi_top_length}" w="${chassi_top_width}" h="${chassi_top_height}"
-                           xyz="0.0 0.0 ${chassi_top_height/2}" rpy="0 0 0"/>
+                           xyz="0.0 0.0 ${chassi_top_height/2}" rpy="0 ${pi/2} 0"/>
     </link>
     <gazebo reference="chassis_top">
@@ -65,22 +65,57 @@
                 <origin xyz="0.0 0.0 0.0" rpy="${pi/2} 0.0 0.0"/>
                 <geometry>
-                    <cylinder radius="${wheel_radius}" length="${wheel_length}"/>
+                    <sphere radius="${wheel_radius}"/>
                 </geometry>
             </collision>
-            <xacro:cylinder_inertia m="0.3" r="${wheel_radius}" h="${wheel_length}"
-                           xyz="0 0 0" rpy="${pi/2} 0.0 0.0"/>
+            <xacro:cylinder_inertia m="0.3" r="${wheel_radius/2}" h="${wheel_length/2}"
+                           xyz="0 0 0" rpy="${pi/2} 0 0"/>
         </link>
         <gazebo reference="${prefix}_wheel">
             <material>Gazebo/Grey</material>
-            <mu1 value="0.1"/>
-            <mu2 value="0.1"/>
+          <!--  <mu1 value="0.1"/>
+            <mu2 value="0.1"/>-->
+            <mu1>100000000000000.0</mu1>
+            <mu2>100000000000000.0</mu2>
+            <kp>1000000000000.0</kp>
+            <kd>10.0</kd>
+            <minDepth>0.001</minDepth>
+            <maxVel>0.1</maxVel>
+            <fdir1>1 0 0</fdir1>
         </gazebo>
     </xacro:macro>
     <xacro:wheel_link prefix="right"/>
     <xacro:wheel_link prefix="left"/>
-    <xacro:wheel_link prefix="right_f"/>
-    <xacro:wheel_link prefix="right_r"/>
-    <xacro:wheel_link prefix="left_f"/>
-    <xacro:wheel_link prefix="left_r"/>
+    <xacro:macro name="caster_wheel_link" params="prefix ">
+        <link name="${prefix}_caster_wheel">
+            <visual>
+                <origin xyz="0.0 0.0 0.0" rpy="${pi/2} 0.0 0.0"/>
+                <geometry>
+                    <cylinder radius="${wheel_radius}" length="${wheel_length}"/>
+                </geometry>
+                <material name="white"/>
+            </visual>
+            <collision>
+                <origin xyz="0.0 0.0 0.0" rpy="${pi/2} 0.0 0.0"/>
+                <geometry>
+                    <sphere radius="${wheel_radius}"/>
+                </geometry>
+            </collision>
+            <xacro:cylinder_inertia m="0.3" r="${wheel_radius/2}" h="${wheel_length/2}"
+                           xyz="0 0 0" rpy="${pi/2} 0 0"/>
+        </link>
+        <gazebo reference="${prefix}_caster_wheel">
+            <material>Gazebo/Grey</material>
+            <mu1>0.01</mu1>
+            <mu2>0.01</mu2>
+            <kp>1000000.0</kp>
+            <kd>100.0</kd>
+            <minDepth>0.001</minDepth>
+            <maxVel>0.1</maxVel>
+        </gazebo>
+    </xacro:macro>
+    <xacro:caster_wheel_link prefix="left_f"/>
+    <xacro:caster_wheel_link prefix="left_r"/>
+    <xacro:caster_wheel_link prefix="right_f"/>
+    <xacro:caster_wheel_link prefix="right_r"/>
     <!-- Joints Fixed -->
     <joint name="base_link" type="fixed">
@@ -99,5 +134,5 @@
         <child link="right_wheel"/>
         <axis xyz="0 1 0"/>
-        <origin xyz="0 -${chassi_width/2 + wheel_length/2} 0" rpy="0 0 0"/>
+        <origin xyz="0 -${chassi_width/2 + wheel_length/2 + 0.005} 0" rpy="0 0 0"/>
     </joint>
     <joint name="joint_2" type="continuous">
@@ -105,32 +140,32 @@
         <child link="left_wheel"/>
         <axis xyz="0 1 0"/>
-        <origin xyz="0 ${chassi_width/2+ wheel_length/2} 0" rpy="0 0 0"/>
+        <origin xyz="0 ${chassi_width/2+ wheel_length/2 + 0.005} 0" rpy="0 0 0"/>
     </joint>
     <joint name="joint_rf" type="continuous">
         <parent link="chassis"/>
-        <child link="right_f_wheel"/>
+        <child link="right_f_caster_wheel"/>
         <axis xyz="0 1 0"/>
-        <origin xyz="${chassi_length/3} -${chassi_width/2 + wheel_length/2} 0" rpy="0 0 0"/>
+        <origin xyz="${chassi_length/3} -${chassi_width/2 + wheel_length/2 + 0.005} 0" rpy="0 0 0"/>
         <mimic joint="joint_1" multiplier="1"/>
     </joint>
     <joint name="joint_rr" type="continuous">
         <parent link="chassis"/>
-        <child link="right_r_wheel"/>
+        <child link="right_r_caster_wheel"/>
         <axis xyz="0 1 0"/>
-        <origin xyz="-${chassi_length/3} -${chassi_width/2 + wheel_length/2} 0" rpy="0 0 0"/>
+        <origin xyz="-${chassi_length/3} -${chassi_width/2 + wheel_length/2 + 0.005} 0" rpy="0 0 0"/>
         <mimic joint="joint_1" multiplier="1"/>
     </joint>
     <joint name="joint_lf" type="continuous">
         <parent link="chassis"/>
-        <child link="left_f_wheel"/>
+        <child link="left_f_caster_wheel"/>
         <axis xyz="0 1 0"/>
-        <origin xyz="${chassi_length/3} ${chassi_width/2 + wheel_length/2} 0" rpy="0 0 0"/>
+        <origin xyz="${chassi_length/3} ${chassi_width/2 + wheel_length/2 + 0.005} 0" rpy="0 0 0"/>
         <mimic joint="joint_2" multiplier="1"/>
     </joint>
     <joint name="joint_lr" type="continuous">
         <parent link="chassis"/>
-        <child link="left_r_wheel"/>
+        <child link="left_r_caster_wheel"/>
         <axis xyz="0 1 0"/>
-        <origin xyz="-${chassi_length/3} ${chassi_width/2 + wheel_length/2} 0" rpy="0 0 0"/>
+        <origin xyz="-${chassi_length/3} ${chassi_width/2 + wheel_length/2 + 0.005} 0" rpy="0 0 0"/>
         <mimic joint="joint_2" multiplier="1"/>
     </joint>

File: tank_description/urdf/leopard.urdf.xacro (robot description, xacro)
@@ -2,10 +2,14 @@
 <robot xmlns:xacro="http://www.ros.org/wiki/xacro" name="leopard">
   <xacro:include filename="material.xacro" />
+  <!--  Chassis Turm und Rohr -->
   <xacro:include filename="chassi.xacro" />
   <xacro:include filename="turret.xacro" />
   <xacro:include filename="pipe.xacro"/>
-<!--
+  <!-- Lidar und Camera
   <xacro:include filename="lidar.xacro" />
   <xacro:include filename="camera.xacro" />
 -->
+  <!-- Gazebo und Ros2 Control-->
+  <xacro:include filename="leopard_gazebo.xacro"/>
+  <xacro:include filename="leopard_ros2_control.xacro"/>
 </robot>

File: tank_description/urdf/pipe.xacro (robot description, xacro)
@@ -14,9 +14,16 @@
             </geometry>
         </collision>
-        <xacro:box_inertia m="0.1" l="0.08" w="0.04" h="0.05"
+        <xacro:box_inertia m="0.1" l="0.008" w="0.004" h="0.005"
                            xyz="0 0 0" rpy="0 0 0"/>
     </link>
     <gazebo reference="turm_gun">
         <material>Gazebo/Grass</material>
+        <mu1>100000000000000.0</mu1>
+        <mu2>100000000000000.0</mu2>
+        <kp>1000000000000.0</kp>
+        <kd>10.0</kd>
+        <minDepth>0.001</minDepth>
+        <maxVel>0.1</maxVel>
+        <fdir1>1 0 0</fdir1>
     </gazebo>
     <link name="gun_deko">
@@ -34,5 +41,5 @@
             </geometry>
         </collision>
-        <xacro:box_inertia m="0.1" l="0.036" w="0.04" h="0.036"
+        <xacro:box_inertia m="0.1" l="0.036" w="0.004" h="0.0036"
                            xyz="0 0 0" rpy="0.0 ${pi/4} 0.0"/>
     </link>
@@ -54,5 +61,5 @@
             </geometry>
         </collision>
-        <xacro:cylinder_inertia m="0.05" r="0.009" h="0.3"
+        <xacro:cylinder_inertia m="0.05" r="0.009" h="0.03"
                            xyz="0.15 0.0 0.0" rpy="0.0 ${pi/2} 0.0"/>
     </link>
@@ -74,5 +81,5 @@
             </geometry>
         </collision>
-        <xacro:cylinder_inertia m="0.001" r="0.00759" h="0.001"
+        <xacro:cylinder_inertia m="0.001" r="0.0075" h="0.001"
                            xyz="0.0 0.0 0.0" rpy="0.0 ${pi/2} 0.0"/>
     </link>

File: tank_description/urdf/turret.xacro (robot description, xacro)
@@ -18,4 +18,14 @@
                            xyz="0 0 0" rpy="0 0 0"/>
         </link>
+        <gazebo reference="${prefix}_coil">
+            <material>Gazebo/Black</material>
+            <mu1>100000000000000.0</mu1>
+            <mu2>100000000000000.0</mu2>
+            <kp>1000000000000.0</kp>
+            <kd>10.0</kd>
+            <minDepth>0.001</minDepth>
+            <maxVel>0.1</maxVel>
+            <fdir1>1 0 0</fdir1>
+        </gazebo>
     </xacro:macro>
     <xacro:turret_coil prefix="top" />
@@ -35,6 +45,6 @@
             <material name="white" />
         </collision>
-        <xacro:box_inertia m="0.5" l="0.28" w="0.17" h="0.05"
-                           xyz="0 0 0" rpy="0 0 0"/>
+        <xacro:box_inertia m="0.5" l="0.02" w="0.01" h="0.05"
+                           xyz="0.06 0 0" rpy="0 0 0"/>
     </link>
     <gazebo reference="turm_top_">
@@ -54,5 +64,5 @@
                 </geometry>
             </collision>
-            <xacro:box_inertia m="0.2" l="0.1" w="0.05" h="0.05"
+            <xacro:box_inertia m="0.2" l="0.005" w="0.0025" h="0.0025"
                            xyz="0 0 0" rpy="0 0 0"/>
         </link>
@@ -74,5 +84,5 @@
                 </geometry>
             </collision>
-            <xacro:box_inertia m="0.1" l="0.0355" w="0.05" h="0.0355"
+            <xacro:box_inertia m="0.1" l="0.00355" w="0.005" h="0.00355"
                                xyz="0 0 0" rpy="0.0 ${pi/4} 0.0"/>
         </link>
@@ -100,9 +110,8 @@
         <child link="top_coil" />
     </joint>  -->
-    <joint name="joint_3" type="revolute">
+    <joint name="joint_3" type="continuous">
         <parent link="down_coil" />
         <child link="top_coil" />
         <axis xyz="0 0 1" />
-        <limit lower="-${pi*2}" upper="${pi*2}" velocity="1.0" effort="10.0" />
         <origin xyz="0 0 0.005" rpy="0 0 0" />
     </joint>
