Commit message: schwachsinn entfernt

File: tank_description/urdf/chassi.xacro (robot description, xacro)
@@ -1,31 +1,31 @@
 <?xml version="1.0"?>
 <robot xmlns:xacro="http://www.ros.org/wiki/xacro">
-    <xacro:property name="chassi_length" value="0.5"/>
-    <xacro:property name="chassi_width" value="0.13"/>
-    <xacro:property name="chassi_height" value="0.06"/>
-    <xacro:property name="chassi_top_length" value="0.5"/>
-    <xacro:property name="chassi_top_width" value="0.23"/>
-    <xacro:property name="chassi_top_height" value="0.04"/>
-    <xacro:property name="wheel_radius" value="0.035"/>
-    <xacro:property name="wheel_length" value="0.028"/>
+    <xacro:property name="chassi_length" value="0.5" />
+    <xacro:property name="chassi_width" value="0.13" />
+    <xacro:property name="chassi_height" value="0.06" />
+    <xacro:property name="chassi_top_length" value="0.5" />
+    <xacro:property name="chassi_top_width" value="0.23" />
+    <xacro:property name="chassi_top_height" value="0.04" />
+    <xacro:property name="wheel_radius" value="0.035" />
+    <xacro:property name="wheel_length" value="0.028" />
     <!-- Links-->
-    <link name="base_footprint"/>
+    <link name="base_footprint" />
     <!-- Chassis Aufbau-->
     <link name="chassis">
         <visual>
-            <origin xyz="0.0 0.0 ${chassi_height/2}" rpy="0.0 0.0 0.0"/>
+            <origin xyz="0.0 0.0 ${chassi_height/2}" rpy="0.0 0.0 0.0" />
             <geometry>
-                <box size="${chassi_length} ${chassi_width} ${chassi_height}"/>
+                <box size="${chassi_length} ${chassi_width} ${chassi_height}" />
             </geometry>
-            <material name="black"/>
+            <material name="black" />
         </visual>
         <collision>
-            <origin xyz="0.0 0.0 ${chassi_height/2}" rpy="0.0 0.0 0.0"/>
+            <origin xyz="0.0 0.0 ${chassi_height/2}" rpy="0.0 0.0 0.0" />
             <geometry>
-                <box size="${chassi_length} ${chassi_width} ${chassi_height}"/>
+                <box size="${chassi_length} ${chassi_width} ${chassi_height}" />
             </geometry>
         </collision>
         <xacro:box_inertia m="3.0" l="${chassi_length}" w="${chassi_width}" h="${chassi_height}"
-                           xyz="0.0 0.0 ${chassi_height/2}" rpy="0 0 0"/>
+            xyz="0.0 0.0 ${chassi_height/2}" rpy="0 0 0" />
     </link>
     <gazebo reference="chassis">
@@ -34,18 +34,19 @@
     <link name="chassis_top">
         <visual>
-            <origin xyz="0.0 0.0 ${chassi_top_height/2}" rpy="0.0 0.0 0.0"/>
+            <origin xyz="0.0 0.0 ${chassi_top_height/2}" rpy="0.0 0.0 0.0" />
             <geometry>
-                <box size="${chassi_top_length} ${chassi_top_width} ${chassi_top_height}"/>
+                <box size="${chassi_top_length} ${chassi_top_width} ${chassi_top_height}" />
             </geometry>
-            <material name="black"/>
+            <material name="black" />
         </visual>
         <collision>
-            <origin xyz="0.0 0.0 ${chassi_top_height/2}" rpy="0.0 0.0 0.0"/>
+            <origin xyz="0.0 0.0 ${chassi_top_height/2}" rpy="0.0 0.0 0.0" />
             <geometry>
-                <box size="${chassi_top_length} ${chassi_top_width} ${chassi_top_height}"/>
+                <box size="${chassi_top_length} ${chassi_top_width} ${chassi_top_height}" />
             </geometry>
         </collision>
-        <xacro:box_inertia m="1.0" l="${chassi_top_length}" w="${chassi_top_width}" h="${chassi_top_height}"
-                           xyz="0.0 0.0 ${chassi_top_height/2}" rpy="0 ${pi/2} 0"/>
+        <xacro:box_inertia m="1.0" l="${chassi_top_length}" w="${chassi_top_width}"
+            h="${chassi_top_height}"
+            xyz="0.0 0.0 ${chassi_top_height/2}" rpy="0 ${pi/2} 0" />
     </link>
     <gazebo reference="chassis_top">
@@ -56,23 +57,21 @@
         <link name="${prefix}_wheel">
             <visual>
-                <origin xyz="0.0 0.0 0.0" rpy="${pi/2} 0.0 0.0"/>
+                <origin xyz="0.0 0.0 0.0" rpy="${pi/2} 0.0 0.0" />
                 <geometry>
-                    <cylinder radius="${wheel_radius}" length="${wheel_length}"/>
+                    <cylinder radius="${wheel_radius}" length="${wheel_length}" />
                 </geometry>
-                <material name="white"/>
+                <material name="white" />
             </visual>
             <collision>
-                <origin xyz="0.0 0.0 0.0" rpy="${pi/2} 0.0 0.0"/>
+                <origin xyz="0.0 0.0 0.0" rpy="${pi/2} 0.0 0.0" />
                 <geometry>
-                    <sphere radius="${wheel_radius}"/>
+                    <sphere radius="${wheel_radius}" />
                 </geometry>
             </collision>
             <xacro:cylinder_inertia m="0.3" r="${wheel_radius/2}" h="${wheel_length/2}"
-                           xyz="0 0 0" rpy="${pi/2} 0 0"/>
+                xyz="0 0 0" rpy="${pi/2} 0 0" />
         </link>
         <gazebo reference="${prefix}_wheel">
             <material>Gazebo/Grey</material>
-          <!--  <mu1 value="0.1"/>
-            <mu2 value="0.1"/>-->
             <mu1>100000000000000.0</mu1>
             <mu2>100000000000000.0</mu2>
@@ -84,23 +83,23 @@
         </gazebo>
     </xacro:macro>
-    <xacro:wheel_link prefix="right"/>
-    <xacro:wheel_link prefix="left"/>
+    <xacro:wheel_link prefix="right" />
+    <xacro:wheel_link prefix="left" />
     <xacro:macro name="caster_wheel_link" params="prefix ">
         <link name="${prefix}_caster_wheel">
             <visual>
-                <origin xyz="0.0 0.0 0.0" rpy="${pi/2} 0.0 0.0"/>
+                <origin xyz="0.0 0.0 0.0" rpy="${pi/2} 0.0 0.0" />
                 <geometry>
-                    <cylinder radius="${wheel_radius}" length="${wheel_length}"/>
+                    <cylinder radius="${wheel_radius}" length="${wheel_length}" />
                 </geometry>
-                <material name="white"/>
+                <material name="white" />
             </visual>
             <collision>
-                <origin xyz="0.0 0.0 0.0" rpy="${pi/2} 0.0 0.0"/>
+                <origin xyz="0.0 0.0 0.0" rpy="${pi/2} 0.0 0.0" />
                 <geometry>
-                    <sphere radius="${wheel_radius}"/>
+                    <sphere radius="${wheel_radius}" />
                 </geometry>
             </collision>
             <xacro:cylinder_inertia m="0.3" r="${wheel_radius/2}" h="${wheel_length/2}"
-                           xyz="0 0 0" rpy="${pi/2} 0 0"/>
+                xyz="0 0 0" rpy="${pi/2} 0 0" />
         </link>
         <gazebo reference="${prefix}_caster_wheel">
@@ -114,59 +113,51 @@
         </gazebo>
     </xacro:macro>
-    <xacro:caster_wheel_link prefix="left_f"/>
-    <xacro:caster_wheel_link prefix="left_r"/>
-    <xacro:caster_wheel_link prefix="right_f"/>
-    <xacro:caster_wheel_link prefix="right_r"/>
+    <xacro:caster_wheel_link prefix="left_f" />
+    <xacro:caster_wheel_link prefix="left_r" />
+    <xacro:caster_wheel_link prefix="right_f" />
+    <xacro:caster_wheel_link prefix="right_r" />
     <!-- Joints Fixed -->
     <joint name="base_link" type="fixed">
-        <parent link="base_footprint"/>
-        <child link="chassis"/>
-        <origin xyz="0.0 0.0 ${wheel_radius}" rpy="0.0 0.0 0.0"/>
+        <parent link="base_footprint" />
+        <child link="chassis" />
+        <origin xyz="0.0 0.0 ${wheel_radius}" rpy="0.0 0.0 0.0" />
     </joint>
     <joint name="chassieAufbau" type="fixed">
-        <parent link="chassis"/>
-        <child link="chassis_top"/>
-        <origin xyz="0.0 0.0 ${chassi_height}" rpy="0.0 0.0 0.0"/>
+        <parent link="chassis" />
+        <child link="chassis_top" />
+        <origin xyz="0.0 0.0 ${chassi_height}" rpy="0.0 0.0 0.0" />
+    </joint>
+    <joint name="joint_rf" type="fixed">
+        <parent link="chassis" />
+        <child link="right_f_caster_wheel" />
+        <origin xyz="${chassi_length/3} -${chassi_width/2 + wheel_length/2 + 0.005} 0" rpy="0 0 0" />
+    </joint>
+    <joint name="joint_rr" type="fixed">
+        <parent link="chassis" />
+        <child link="right_r_caster_wheel" />
+        <origin xyz="-${chassi_length/3} -${chassi_width/2 + wheel_length/2 + 0.005} 0" rpy="0 0 0" />
+    </joint>
+    <joint name="joint_lf" type="fixed">
+        <parent link="chassis" />
+        <child link="left_f_caster_wheel" />
+        <origin xyz="${chassi_length/3} ${chassi_width/2 + wheel_length/2 + 0.005} 0" rpy="0 0 0" />
+    </joint>
+    <joint name="joint_lr" type="fixed">
+        <parent link="chassis" />
+        <child link="left_r_caster_wheel" />
+        <origin xyz="-${chassi_length/3} ${chassi_width/2 + wheel_length/2 + 0.005} 0" rpy="0 0 0" />
     </joint>
     <!-- Joints Moving-->
     <joint name="joint_1" type="continuous">
-        <parent link="chassis"/>
-        <child link="right_wheel"/>
-        <axis xyz="0 1 0"/>
-        <origin xyz="0 -${chassi_width/2 + wheel_length/2 + 0.005} 0" rpy="0 0 0"/>
+        <parent link="chassis" />
+        <child link="right_wheel" />
+        <axis xyz="0 1 0" />
+        <origin xyz="0 -${chassi_width/2 + wheel_length/2 + 0.005} 0" rpy="0 0 0" />
     </joint>
     <joint name="joint_2" type="continuous">
-        <parent link="chassis"/>
-        <child link="left_wheel"/>
-        <axis xyz="0 1 0"/>
-        <origin xyz="0 ${chassi_width/2+ wheel_length/2 + 0.005} 0" rpy="0 0 0"/>
-    </joint>
-    <joint name="joint_rf" type="continuous">
-        <parent link="chassis"/>
-        <child link="right_f_caster_wheel"/>
-        <axis xyz="0 1 0"/>
-        <origin xyz="${chassi_length/3} -${chassi_width/2 + wheel_length/2 + 0.005} 0" rpy="0 0 0"/>
-        <mimic joint="joint_1" multiplier="1"/>
-    </joint>
-    <joint name="joint_rr" type="continuous">
-        <parent link="chassis"/>
-        <child link="right_r_caster_wheel"/>
-        <axis xyz="0 1 0"/>
-        <origin xyz="-${chassi_length/3} -${chassi_width/2 + wheel_length/2 + 0.005} 0" rpy="0 0 0"/>
-        <mimic joint="joint_1" multiplier="1"/>
-    </joint>
-    <joint name="joint_lf" type="continuous">
-        <parent link="chassis"/>
-        <child link="left_f_caster_wheel"/>
-        <axis xyz="0 1 0"/>
-        <origin xyz="${chassi_length/3} ${chassi_width/2 + wheel_length/2 + 0.005} 0" rpy="0 0 0"/>
-        <mimic joint="joint_2" multiplier="1"/>
-    </joint>
-    <joint name="joint_lr" type="continuous">
-        <parent link="chassis"/>
-        <child link="left_r_caster_wheel"/>
-        <axis xyz="0 1 0"/>
-        <origin xyz="-${chassi_length/3} ${chassi_width/2 + wheel_length/2 + 0.005} 0" rpy="0 0 0"/>
-        <mimic joint="joint_2" multiplier="1"/>
+        <parent link="chassis" />
+        <child link="left_wheel" />
+        <axis xyz="0 1 0" />
+        <origin xyz="0 ${chassi_width/2+ wheel_length/2 + 0.005} 0" rpy="0 0 0" />
     </joint>
 </robot>

File: tank_description/urdf/leopard_ros2_control.xacro (robot description, xacro)
@@ -7,36 +7,4 @@
                 <plugin>gazebo_ros2_control/GazeboSystem</plugin>
             </hardware>
-            <joint name="joint_lf">
-                <param name="mimic">joint_2</param>
-                <param name="multiplier">-1</param>
-                <command_interface name="velocity">
-                    <parma name="min">-1</parma>
-                    <parma name="max">1</parma>
-                </command_interface>
-            </joint>
-            <joint name="joint_lr">
-                <param name="mimic">joint_2</param>
-                <param name="multiplier">-1</param>
-                <command_interface name="velocity">
-                    <parma name="min">-1</parma>
-                    <parma name="max">1</parma>
-                </command_interface>
-            </joint>
-            <joint name="joint_rf">
-                <param name="mimic">joint_1</param>
-                <param name="multiplier">-1</param>
-                <command_interface name="velocity">
-                    <parma name="min">-1</parma>
-                    <parma name="max">1</parma>
-                </command_interface>
-            </joint>
-            <joint name="joint_rr">
-                <param name="mimic">joint_1</param>
-                <param name="multiplier">-1</param>
-                <command_interface name="velocity">
-                    <parma name="min">-1</parma>
-                    <parma name="max">1</parma>
-                </command_interface>
-            </joint>
         </xacro:if>
         <xacro:unless value="$(arg is_sim)">
@@ -80,36 +48,4 @@
             <state_interface name="position" />
         </joint>
-        <joint name="joint_lf">
-            <param name="mimic">joint_2</param>
-            <param name="multiplier">1</param>
-            <command_interface name="velocity">
-                <parma name="min">-1</parma>
-                <parma name="max">1</parma>
-            </command_interface>
-        </joint>
-        <joint name="joint_lr">
-            <param name="mimic">joint_2</param>
-            <param name="multiplier">1</param>
-            <command_interface name="velocity">
-                <parma name="min">-1</parma>
-                <parma name="max">1</parma>
-            </command_interface>
-        </joint>
-        <joint name="joint_rf">
-            <param name="mimic">joint_1</param>
-            <param name="multiplier">1</param>
-            <command_interface name="velocity">
-                <parma name="min">-1</parma>
-                <parma name="max">1</parma>
-            </command_interface>
-        </joint>
-        <joint name="joint_rr">
-            <param name="mimic">joint_1</param>
-            <param name="multiplier">1</param>
-            <command_interface name="velocity">
-                <parma name="min">-1</parma>
-                <parma name="max">1</parma>
-            </command_interface>
-        </joint>
     </ros2_control>
 </robot>
