Commit message: in work

File: tank_description/urdf/leopard_ros2_control.xacro (robot description, xacro)
@@ -35,12 +35,4 @@
                 <plugin>gazebo_ros2_control/GazeboSystem</plugin>
             </hardware>
-            <joint name="joint_4">
-                <command_interface name="velocity">
-                    <parma name="min">-1</parma>
-                    <parma name="max">1</parma>
-                </command_interface>
-                <state_interface name="position" />
-                <state_interface name="velocity" />
-            </joint>
         </xacro:if>
         <xacro:unless value="$(arg is_sim)">
@@ -58,4 +50,12 @@
             <state_interface name="velocity" />
         </joint>
+        <joint name="joint_4">
+            <command_interface name="velocity">
+                <parma name="min">-1</parma>
+                <parma name="max">1</parma>
+            </command_interface>
+            <state_interface name="position" />
+            <state_interface name="velocity" />
+        </joint>
     </ros2_control>
     <!--
