Commit message: in work

File: tank_description/urdf/leopard.urdf.xacro (robot description, xacro)
@@ -1,10 +1,11 @@
 <?xml version="1.0"?>
 <robot xmlns:xacro="http://www.ros.org/wiki/xacro" name="leopard">
+  <xacro:arg name="is_sim" default="true"/>
   <xacro:include filename="material.xacro" />
   <!--  Chassis Turm und Rohr -->
   <xacro:include filename="chassi.xacro" />
-  <xacro:include filename="turret.xacro" />
+<!--   <xacro:include filename="turret.xacro" />
   <xacro:include filename="pipe.xacro"/>
-  <!-- Lidar und Camera
+  Lidar und Camera
   <xacro:include filename="lidar.xacro" />
   <xacro:include filename="camera.xacro" />

File: tank_description/urdf/leopard_gazebo.xacro (robot description, xacro)
@@ -19,22 +19,4 @@
         </joint>
     </transmission>
-    <transmission name="turret_transmission" >
-        <plugin>
-            transmission_interface/SimpleTransmission
-        </plugin>
-        <actuator name="turret_motor" role="actuator_turret" />
-        <joint name="joint_3" role="joint_rotate" >
-            <mechanical_reduction>1.0</mechanical_reduction>
-        </joint>
-    </transmission>
-    <transmission name="pipe_transmission" >
-        <plugin>
-            transmission_interface/SimpleTransmission
-        </plugin>
-        <actuator name="pipe_motor" role="actuator_pipe" />
-        <joint name="joint_4" role="joint_lift" >
-            <mechanical_reduction>1.0</mechanical_reduction>
-        </joint>
-    </transmission>
     <gazebo>
         <plugin filename="libgazebo_ros2_control.so" name="gazebo_ros2_control">

File: tank_description/urdf/leopard_ros2_control.xacro (robot description, xacro)
@@ -2,5 +2,4 @@
 <robot xmlns:xacro="http://www.ros.org/wiki/xacro">
     <ros2_control type="system" name="PanzerSystem">
-<!--
         <xacro:if value="$(arg is_sim)">
             <hardware>
@@ -10,12 +9,8 @@
         <xacro:unless value="$(arg is_sim)">
             <hardware>
-                <plugin>leopard_firmware/TankInterface</plugin>
+                <plugin>chassis_firmware/ChassisInterface</plugin>
                 <param name="port">/dev/ttyUSB0</param>
             </hardware>
         </xacro:unless>
-    -->
-        <hardware>
-            <plugin>gazebo_ros2_control/GazeboSystem</plugin>
-        </hardware>
         <joint name="joint_1">
             <command_interface name="velocity">
@@ -34,4 +29,5 @@
             <state_interface name="velocity" />
         </joint>
+<!--
         <joint name="joint_3">
             <command_interface name="velocity">
@@ -50,4 +46,5 @@
             <state_interface name="velocity" />
         </joint>
+    -->
     </ros2_control>
 </robot>

File: tank_description/urdf/pipe.xacro (robot description, xacro)
@@ -116,3 +116,12 @@
         <origin xyz="0.3005 0.0 0.0" rpy="0.0 0.0 0.0" />
     </joint>
+    <transmission name="pipe_transmission" >
+        <plugin>
+            transmission_interface/SimpleTransmission
+        </plugin>
+        <actuator name="pipe_motor" role="actuator_pipe" />
+        <joint name="joint_4" role="joint_lift" >
+            <mechanical_reduction>1.0</mechanical_reduction>
+        </joint>
+    </transmission>
 </robot>

File: tank_description/urdf/turret.xacro (robot description, xacro)
@@ -132,3 +132,12 @@
         <origin xyz="0.17 -0.06 0.0" />
     </joint>
+    <transmission name="turret_transmission" >
+        <plugin>
+            transmission_interface/SimpleTransmission
+        </plugin>
+        <actuator name="turret_motor" role="actuator_turret" />
+        <joint name="joint_3" role="joint_rotate" >
+            <mechanical_reduction>1.0</mechanical_reduction>
+        </joint>
+    </transmission>
 </robot>

Commit message: turret hardware interface in work

File: tank_description/urdf/leopard.urdf.xacro (robot description, xacro)
@@ -5,6 +5,6 @@
   <!--  Chassis Turm und Rohr -->
   <xacro:include filename="chassi.xacro" />
-<!--   <xacro:include filename="turret.xacro" />
-  <xacro:include filename="pipe.xacro"/>
+  <xacro:include filename="turret.xacro" />
+<!--  <xacro:include filename="pipe.xacro"/>
   Lidar und Camera
   <xacro:include filename="lidar.xacro" />

File: tank_description/urdf/leopard_ros2_control.xacro (robot description, xacro)
@@ -30,5 +30,4 @@
         </joint>
     </ros2_control>
-<!--
     <ros2_control type="system" name="Turret_System">
         <xacro:if value="$(arg is_sim)">
@@ -51,5 +50,7 @@
             <state_interface name="velocity" />
         </joint>
-        <joint name="joint_4">
+    </ros2_control>
+    <!--
+    <joint name="joint_4">
             <command_interface name="velocity">
                 <parma name="min">-1</parma>
@@ -59,4 +60,4 @@
             <state_interface name="velocity" />
         </joint>
-    </ros2_control> -->
+        -->
 </robot>

Commit message: controller works

File: tank_description/urdf/leopard.urdf.xacro (robot description, xacro)
@@ -6,6 +6,6 @@
   <xacro:include filename="chassi.xacro" />
   <xacro:include filename="turret.xacro" />
-<!--  <xacro:include filename="pipe.xacro"/>
-  Lidar und Camera
+  <xacro:include filename="pipe.xacro"/>
+  <!-- Lidar und Camera
   <xacro:include filename="lidar.xacro" />
   <xacro:include filename="camera.xacro" />

File: tank_description/urdf/leopard_ros2_control.xacro (robot description, xacro)
@@ -35,4 +35,12 @@
                 <plugin>gazebo_ros2_control/GazeboSystem</plugin>
             </hardware>
+            <joint name="joint_4">
+                <command_interface name="velocity">
+                    <parma name="min">-1</parma>
+                    <parma name="max">1</parma>
+                </command_interface>
+                <state_interface name="position" />
+                <state_interface name="velocity" />
+            </joint>
         </xacro:if>
         <xacro:unless value="$(arg is_sim)">
@@ -52,12 +60,4 @@
     </ros2_control>
     <!--
-    <joint name="joint_4">
-            <command_interface name="velocity">
-                <parma name="min">-1</parma>
-                <parma name="max">1</parma>
-            </command_interface>
-            <state_interface name="position" />
-            <state_interface name="velocity" />
-        </joint>
         -->
 </robot>

Commit message: in work

File: tank_description/urdf/leopard.urdf.xacro (robot description, xacro)
@@ -5,6 +5,5 @@
   <!--  Chassis Turm und Rohr -->
   <xacro:include filename="chassi.xacro" />
-  <!--
-  <xacro:include filename="turret.xacro" />
+  <xacro:include filename="turret.xacro" />  <!--
   <xacro:include filename="pipe.xacro"/>
 -->

File: tank_description/urdf/leopard_ros2_control.xacro (robot description, xacro)
@@ -30,5 +30,4 @@
         </joint>
     </ros2_control>
-<!--
     <ros2_control type="system" name="Turret_System">
         <xacro:if value="$(arg is_sim)">
@@ -44,5 +43,5 @@
         </xacro:unless>
         <joint name="joint_3">
-            <command_interface name="velocity">
+            <command_interface name="position">
                 <parma name="min">-1</parma>
                 <parma name="max">1</parma>
@@ -52,5 +51,4 @@
         </joint>
     </ros2_control>
--->
 <!--
     <ros2_control type="system" name="Pipe_System">

File: tank_description/urdf/turret.xacro (robot description, xacro)
@@ -104,10 +104,4 @@
         <child link="down_coil" />
     </joint>
-    <!-- change to moving if - joint für den turm
-    <joint name="turret_coil_joint" type="fixed">
-        <origin xyz="0.0 0.0 0.005" rpy="0.0 0.0 0.0" />
-        <parent link="down_coil" />
-        <child link="top_coil" />
-    </joint>  -->
     <joint name="joint_3" type="continuous">
         <parent link="down_coil" />

Commit message: only chassis under control

File: tank_description/urdf/leopard.urdf.xacro (robot description, xacro)
@@ -5,5 +5,5 @@
   <!--  Chassis Turm und Rohr -->
   <xacro:include filename="chassi.xacro" />
-  <xacro:include filename="turret.xacro" />  <!--
+  <!--  <xacro:include filename="turret.xacro" />
   <xacro:include filename="pipe.xacro"/>
 -->

File: tank_description/urdf/leopard_ros2_control.xacro (robot description, xacro)
@@ -30,47 +30,3 @@
         </joint>
     </ros2_control>
-    <ros2_control type="system" name="Turret_System">
-        <xacro:if value="$(arg is_sim)">
-            <hardware>
-                <plugin>gazebo_ros2_control/GazeboSystem</plugin>
-            </hardware>
-        </xacro:if>
-        <xacro:unless value="$(arg is_sim)">
-            <hardware>
-                <plugin>turret_firmware/TurretInterface</plugin>
-                <param name="port">/dev/ttyUSB1</param>
-            </hardware>
-        </xacro:unless>
-        <joint name="joint_3">
-            <command_interface name="velocity">
-                <parma name="min">-1</parma>
-                <parma name="max">1</parma>
-            </command_interface>
-            <state_interface name="position" />
-            <state_interface name="velocity" />
-        </joint>
-    </ros2_control>
-<!--
-    <ros2_control type="system" name="Pipe_System">
-        <xacro:if value="$(arg is_sim)">
-            <hardware>
-                <plugin>gazebo_ros2_control/GazeboSystem</plugin>
-            </hardware>
-        </xacro:if>
-        <xacro:unless value="$(arg is_sim)">
-            <hardware>
-                <plugin>pipe_firmware/PipeInterface</plugin>
-                <param name="port">/dev/ttyUSB2</param>
-            </hardware>
-        </xacro:unless>
-        <joint name="joint_4">
-            <command_interface name="velocity">
-                <parma name="min">-1</parma>
-                <parma name="max">1</parma>
-            </command_interface>
-            <state_interface name="position" />
-            <state_interface name="velocity" />
-        </joint>
-    </ros2_control>
--->
 </robot>

File: tank_description/urdf/pipe.xacro (robot description, xacro)
@@ -125,3 +125,26 @@
         </joint>
     </transmission>
+    <!--
+    <ros2_control type="system" name="Pipe_System">
+        <xacro:if value="$(arg is_sim)">
+            <hardware>
+                <plugin>gazebo_ros2_control/GazeboSystem</plugin>
+            </hardware>
+        </xacro:if>
+        <xacro:unless value="$(arg is_sim)">
+            <hardware>
+                <plugin>pipe_firmware/PipeInterface</plugin>
+                <param name="port">/dev/ttyUSB2</param>
+            </hardware>
+        </xacro:unless>
+        <joint name="joint_4">
+            <command_interface name="velocity">
+                <parma name="min">-1</parma>
+                <parma name="max">1</parma>
+            </command_interface>
+            <state_interface name="position" />
+            <state_interface name="velocity" />
+        </joint>
+    </ros2_control>
+-->
 </robot>

File: tank_description/urdf/turret.xacro (robot description, xacro)
@@ -135,3 +135,24 @@
         </joint>
     </transmission>
+    <ros2_control type="system" name="Turret_System">
+        <xacro:if value="$(arg is_sim)">
+            <hardware>
+                <plugin>gazebo_ros2_control/GazeboSystem</plugin>
+            </hardware>
+        </xacro:if>
+        <xacro:unless value="$(arg is_sim)">
+            <hardware>
+                <plugin>turret_firmware/TurretInterface</plugin>
+                <param name="port">/dev/ttyUSB1</param>
+            </hardware>
+        </xacro:unless>
+        <joint name="joint_3">
+            <command_interface name="velocity">
+                <parma name="min">-1</parma>
+                <parma name="max">1</parma>
+            </command_interface>
+            <state_interface name="position" />
+            <state_interface name="velocity" />
+        </joint>
+    </ros2_control>
 </robot>
